File: Project/AISReceiver.sch (KiCad schematic (older format))
At the start: 72 parts, among them J1 SPI, J2 CONN_01X20, J3 CONN_01X20, J4 USB_OTG, P1 Antenna, Q1 2.5A/30V, Q2 MBT3904DW1, SW1 RESET, SW2 BUFFER_RESET, U1 ESP32-WROOM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

Commit message: AIS specific board.
Parts:
- removed C6, C8: 4.7uF, Capacitors_SMD:C_0603_HandSoldering, symbol C_Small
- removed C7: 10uF, Capacitors_SMD:C_0805_HandSoldering, symbol CP_Small
- removed C9: 0.1uF, Capacitors_SMD:C_0603_HandSoldering, symbol C_Small
- removed D3: RED, Pin_Headers:Pin_Header_Straight_1x02_Pitch2.54mm, symbol LED_ALT
- removed D4: BLUE, Pin_Headers:Pin_Header_Straight_1x02_Pitch2.54mm, symbol LED_ALT
- removed JP2: Jumper, Capacitors_SMD:C_0603, symbol Jumper
- removed LIPO1: JP2, Connectors_JST:JST_EH_S02B-EH_02x2.50mm_Angled, symbol CONN_01X02
- removed Q1: 2.5A/30V, TO_SOT_Packages_SMD:SOT-23_Handsoldering, symbol Q_PMOS_SGD
- removed R10, R12: 1K, Resistors_SMD:R_0603_HandSoldering, symbol R_Small
- removed R13, R14: 2K, Resistors_SMD:R_0603_HandSoldering, symbol R_Small
- removed R6, R7: 4.7K, Resistors_SMD:R_0603_HandSoldering, symbol R
- removed R8: 100R, Resistors_SMD:R_0603_HandSoldering, symbol R
- removed R9: 10K, Resistors_SMD:R_0603_HandSoldering, symbol R
- removed U3: MCP73811T-420I/OT, TO_SOT_Packages_SMD:SOT-23-5, symbol MCP73811T-420I/OT
- removed U4: LIS331HH, Si4464:LGA-16-3x3, symbol LIS331HH
- added H1, H2, H3, H4, H5, H6: MountingHole_Pad, Mounting_Wuerth:Mounting_Wuerth_WA-SMSI-M1.6_H1.5mm_9774015633, symbol Mechanical:MountingHole_Pad
- added J5: RF_Shield, RF_Shielding:Wuerth_36103205_20x20mm, symbol Device:RF_Shield_One_Piece
- C1, C19, C2, C20, C3, C4, C5: footprint Capacitors_SMD:C_0603_HandSoldering -> Capacitor_SMD:C_0603_1608Metric_Pad1.08x0.95mm_HandSolder; symbol C_Small -> AISReceiver-rescue:C_Small
- C10, C11, C12, C13, C14, C15: footprint Capacitors_SMD:C_0603_HandSoldering -> Capacitor_SMD:C_0603_1608Metric_Pad1.08x0.95mm_HandSolder; symbol C -> AISReceiver-rescue:C
- C16, C17, C18, CR1, CR2: footprint Capacitors_SMD:C_0603_HandSoldering -> Capacitor_SMD:C_0603_1608Metric_Pad1.08x0.95mm_HandSolder; symbol C-RESCUE-AISReceiver -> AISReceiver-rescue:C-RESCUE-AISReceiver
- CR3: footprint Capacitors_SMD:C_1210_HandSoldering -> Capacitor_SMD:C_1210_3225Metric_Pad1.33x2.70mm_HandSolder; symbol C-RESCUE-AISReceiver -> AISReceiver-rescue:C-RESCUE-AISReceiver
- D1: footprint Si4464:SOD-323 -> Diode_SMD:D_SOD-323; symbol BAT48JFILM -> AISReceiver-rescue:BAT48JFILM
- D2, D5: footprint Pin_Headers:Pin_Header_Straight_1x02_Pitch2.54mm -> LED_THT:LED_D3.0mm_Clear; symbol LED_ALT -> AISReceiver-rescue:LED_ALT
- F1: footprint Fuse_Holders_and_Fuses:Fuse_SMD1206_Wave -> Fuses:1206; symbol Polyfuse -> AISReceiver-rescue:Polyfuse
- J1: footprint Pin_Headers:Pin_Header_Angled_2x03_Pitch2.54mm -> Connector_PinHeader_2.54mm:PinHeader_2x03_P2.54mm_Horizontal; symbol CONN_02X03 -> AISReceiver-rescue:CONN_02X03
- J2, J3: footprint Pin_Headers:Pin_Header_Straight_1x20_Pitch2.54mm -> Connector_PinHeader_2.54mm:PinHeader_2x10_P2.54mm_Vertical; symbol CONN_01X20 -> AISReceiver-rescue:CONN_01X20
- J4: symbol USB_OTG -> AISReceiver-rescue:USB_OTG
- JP1: footprint Capacitors_SMD:C_0603 -> Capacitor_SMD:C_0603_1608Metric_Pad1.08x0.95mm_HandSolder; symbol Jumper -> AISReceiver-rescue:Jumper
- LR1: footprint Capacitors_SMD:C_0805_HandSoldering -> Capacitor_SMD:C_0805_2012Metric_Pad1.18x1.45mm_HandSolder; symbol INDUCTOR -> AISReceiver-rescue:INDUCTOR
- LR2: footprint Capacitors_SMD:C_0402 -> Capacitor_SMD:C_0402_1005Metric_Pad0.74x0.62mm_HandSolder; symbol INDUCTOR -> AISReceiver-rescue:INDUCTOR
- P1: footprint Connectors_Molex:Molex_Microcoaxial_RF -> Connector_Coaxial:SMA_Amphenol_132134_Vertical; symbol BNC -> AISReceiver-rescue:BNC
- Q2: symbol MBT3904DW1 -> AISReceiver-rescue:MBT3904DW1
- R1, R11, R15, R16, R17, R18, R19, R2, R21, R3: footprint Resistors_SMD:R_0603_HandSoldering -> Resistor_SMD:R_0603_1608Metric_Pad0.98x0.95mm_HandSolder; symbol R -> AISReceiver-rescue:R
- R20, R22: footprint Resistors_SMD:R_0603_HandSoldering -> Resistor_SMD:R_0603_1608Metric_Pad0.98x0.95mm_HandSolder; symbol R-RESCUE-AISReceiver -> AISReceiver-rescue:R-RESCUE-AISReceiver
- R4, R5: footprint Resistors_SMD:R_0603_HandSoldering -> Resistor_SMD:R_0603_1608Metric_Pad0.98x0.95mm_HandSolder; symbol R_Small -> AISReceiver-rescue:R_Small
- SW1, SW2: footprint Buttons_Switches_SMD:SW_SPST_B3SL-1002P -> Button_Switch_SMD:SW_SPST_B3SL-1022P; symbol SW_Push -> AISReceiver-rescue:SW_Push
- U1: footprint ESP32-footprints-Lib:ESP32-WROOM -> RF_Module:ESP32-WROOM-32; symbol ESP32-WROOM -> AISReceiver-rescue:ESP32-WROOM
- U2: footprint TO_SOT_Packages_SMD:SOT-23-5 -> Package_TO_SOT_SMD:SOT-23-5_HandSoldering; symbol AP131-35 -> AISReceiver-rescue:AP131-35
- U5: footprint SMD_Packages:SSOP-20 -> Silicon-Standard:SSOP_20; symbol FT231XS -> AISReceiver-rescue:FT231XS
- U6: symbol Si4362 -> AISReceiver-rescue:Si4362
- X1: footprint Crystals:Crystal_SMD_0603-4pin_6.0x3.5mm_HandSoldering -> Crystal:Crystal_SMD_0603-4Pin_6.0x3.5mm_HandSoldering; symbol Crystal_GND23 -> AISReceiver-rescue:Crystal_GND23
Connections:
- net GND: now also H1.1, H2.1, H3.1, H4.1, H5.1, H6.1, J5.1 (Shield)
- net V_BATT: no longer names the net of J2.3 (P3)
- net V_BATT: no longer J3.3 (P3)
Other:
- note removed: "3.3V LI-PO BATTERY CHARGER"
- note removed: "ACCELEROMETER"
